Commit message: removed pybullet_envs requirement

File: pmtg/gym-hsa_robot/gym_hsa_robot/resources/hsa_turtle.urdf (robot description, URDF)
Before this commit: robot hsarobot, 7 links, 6 joints
Links:
- removed link left_back_wheel
- removed link left_front_leg
- removed link left_hinge
- removed link right_back_wheel
- removed link right_front_wheel
- removed link right_hinge
- added link dummy, mass 0.001
- added link foot_fl, mass 0.25; collision box size=0.035 0.035 0.02; visual box size=0.035 0.035 0.02
- added link foot_fr, mass 0.25; collision box size=0.035 0.035 0.02; visual box size=0.035 0.035 0.02
- added link foot_rl, mass 0.25; collision box size=0.035 0.035 0.02; visual box size=0.035 0.035 0.02
- added link foot_rr, mass 0.25; collision box size=0.035 0.035 0.02; visual box size=0.035 0.035 0.02
- added link leg_fl, mass 0.02; collision box size=0.035 0.035 0.05; visual box size=0.035 0.035 0.05
- added link leg_fr, mass 0.02; collision box size=0.035 0.035 0.05; visual box size=0.035 0.035 0.05
- added link leg_rl, mass 0.02; collision box size=0.035 0.035 0.05; visual box size=0.035 0.035 0.05
- added link leg_rr, mass 0.02; collision box size=0.035 0.035 0.05; visual box size=0.035 0.035 0.05
- link base_link: mass 0.4 -> 0.01; geometry collision box size=0.14 0.16 0.02; visual box size=0.14 0.16 0.02
Joints:
- removed joint base_to_left_back_wheel
- removed joint base_to_left_hinge
- removed joint base_to_right_back_wheel
- removed joint base_to_right_hinge
- removed joint left_hinge_to_left_front_wheel
- removed joint right_hinge_to_right_front_wheel
- added joint base_to_leg_fl: type revolute, parent base_link, child leg_fl, origin xyz=0.035 0.06 -0.01 rpy=0 0 0, axis 0 1 0, limit lower=-0.23 upper=0.23 effort=10 velocity=1.0
- added joint base_to_leg_fr: type revolute, parent base_link, child leg_fr, origin xyz=0.035 -0.06 -0.01 rpy=0 0 0, axis 0 1 0, limit lower=-0.23 upper=0.23 effort=10 velocity=1.0
- added joint base_to_leg_rl: type revolute, parent base_link, child leg_rl, origin xyz=-0.035 0.06 -0.01 rpy=0 0 0, axis 0 1 0, limit lower=-0.23 upper=0.23 effort=10 velocity=1.0
- added joint base_to_leg_rr: type revolute, parent base_link, child leg_rr, origin xyz=-0.035 -0.06 -0.01 rpy=0 0 0, axis 0 1 0, limit lower=-0.23 upper=0.23 effort=10 velocity=1.0
- added joint dummy_joint: type fixed, parent dummy, child base_link
- added joint leg_to_foot_fl: type prismatic, parent leg_fl, child foot_fl, origin xyz=0.0 0.0 -0.06 rpy=0 0 0, axis 0 0 1, limit lower=-0.008 upper=0.0005 effort=10 velocity=1.0
- added joint leg_to_foot_fr: type prismatic, parent leg_fr, child foot_fr, origin xyz=0.0 0.0 -0.06 rpy=0 0 0, axis 0 0 1, limit lower=-0.008 upper=0.0005 effort=10 velocity=1.0
- added joint leg_to_foot_rl: type prismatic, parent leg_rl, child foot_rl, origin xyz=0.0 0.0 -0.06 rpy=0 0 0, axis 0 0 1, limit lower=-0.008 upper=0.0005 effort=10 velocity=1.0
- added joint leg_to_foot_rr: type prismatic, parent leg_rr, child foot_rr, origin xyz=0.0 0.0 -0.06 rpy=0 0 0, axis 0 0 1, limit lower=-0.008 upper=0.0005 effort=10 velocity=1.0

File: pmtg/gym-hsa_robot/gym_hsa_robot/resources/hsa_turtle.xacro (robot description, xacro)
@@ -123,8 +123,8 @@
             <inertial>
                 <origin rpy="0 0 0" xyz="${leg_x} ${leg_y} -0.06"/>
-                <mass value = "0.01"/>
-                <inertia ixx="${(1.0/12.0) * 0.01 * ( (0.035 * 0.035) + (0.01 * 0.01) ) }"
-                                 iyy="${(1.0/12.0) * 0.01 * ( (0.035 * 0.035) + (0.01 * 0.01) ) }"
-                                 izz="${(1.0/12.0) * 0.01 * ( (0.035 * 0.035) + (0.035 * 0.035) ) }"
+                <mass value = "${foot_mass}"/>
+                <inertia ixx="${(1.0/12.0) * foot_mass * ( (0.035 * 0.035) + (0.01 * 0.01) ) }"
+                                 iyy="${(1.0/12.0) * foot_mass * ( (0.035 * 0.035) + (0.01 * 0.01) ) }"
+                                 izz="${(1.0/12.0) * foot_mass * ( (0.035 * 0.035) + (0.035 * 0.035) ) }"
                                  ixy="0"
                                  ixz="0"
@@ -147,5 +147,5 @@
             <child link="${link_child}" />
                     <!-- What to set these to? -->
-            <limit velocity="1.0" effort="10" lower="-0.3" upper="0.3"/>
+            <limit velocity="1.0" effort="10" lower="-0.23" upper="0.23"/>
         </joint>
     </xacro:macro>
@@ -157,5 +157,5 @@
             <child link="${link_child}" />
                     <!-- What to set these to? -->
-            <limit velocity="1.0" effort="10" lower="-0.02" upper="0.0199"/>
+            <limit velocity="1.0" effort="10" lower="-0.008" upper="0.0005"/>
         </joint>
     </xacro:macro>

File: pmtg/gym-hsa_robot/gym_hsa_robot/resources/hsa_turtle_test.urdf (robot description, URDF)
Before this commit: robot hsa_robot, 10 links, 9 joints
Links:
- link base_link: mass 0.4 -> 0.01
- link foot_fl: mass 0.01 -> 0.25
- link foot_fr: mass 0.01 -> 0.25
- link foot_rl: mass 0.01 -> 0.25
- link foot_rr: mass 0.01 -> 0.25
Joints:
- joint base_to_leg_fl: limit lower=-0.5 upper=0.5 effort=10 velocity=1.0 -> lower=-0.23 upper=0.23 effort=10 velocity=1.0
- joint base_to_leg_fr: limit lower=-0.5 upper=0.5 effort=10 velocity=1.0 -> lower=-0.23 upper=0.23 effort=10 velocity=1.0
- joint base_to_leg_rl: limit lower=-0.5 upper=0.5 effort=10 velocity=1.0 -> lower=-0.23 upper=0.23 effort=10 velocity=1.0
- joint base_to_leg_rr: limit lower=-0.5 upper=0.5 effort=10 velocity=1.0 -> lower=-0.23 upper=0.23 effort=10 velocity=1.0
- joint leg_to_foot_fl: limit lower=-0.02 upper=0.0199 effort=10 velocity=1.0 -> lower=-0.008 upper=0.0005 effort=10 velocity=1.0
- joint leg_to_foot_fr: limit lower=-0.02 upper=0.0199 effort=10 velocity=1.0 -> lower=-0.008 upper=0.0005 effort=10 velocity=1.0
- joint leg_to_foot_rl: limit lower=-0.02 upper=0.0199 effort=10 velocity=1.0 -> lower=-0.008 upper=0.0005 effort=10 velocity=1.0
- joint leg_to_foot_rr: limit lower=-0.02 upper=0.0199 effort=10 velocity=1.0 -> lower=-0.008 upper=0.0005 effort=10 velocity=1.0
