Commit message: xacro changes

File: pmtg/gym-hsa_robot/gym_hsa_robot/resources/hsa_turtle.xacro (robot description, xacro)
@@ -15,12 +15,12 @@
     <xacro:property name="foot_depth" value="0.01" />
 	<xacro:property name="foot_mass" value="0.25" />
-    <xacro:property name="leg_fl_x" value="0.4" />
-    <xacro:property name="leg_fl_y" value="0.4" />
-    <xacro:property name="leg_fr_x" value="0.4" />
-    <xacro:property name="leg_fr_y" value="0.4" />
-    <xacro:property name="leg_rl_x" value="0.4" />
-    <xacro:property name="leg_rl_y" value="0.4" />
-    <xacro:property name="leg_rr_x" value="0.4" />
-    <xacro:property name="leg_rr_y" value="0.4" />
+    <xacro:property name="leg_fl_x" value="0.035" />
+    <xacro:property name="leg_fl_y" value="0.06" />
+    <xacro:property name="leg_fr_x" value="0.035" />
+    <xacro:property name="leg_fr_y" value="-0.06" />
+    <xacro:property name="leg_rl_x" value="-0.035" />
+    <xacro:property name="leg_rl_y" value="0.06" />
+    <xacro:property name="leg_rr_x" value="-0.035" />
+    <xacro:property name="leg_rr_y" value="-0.06" />
     <xacro:property name="foot_fl_x" value="0.4" />
     <xacro:property name="foot_fl_y" value="0.4" />
@@ -104,8 +104,8 @@
         </link>
     </xacro:macro>
-    <xacro:macro name="leg_joint" params="link_child name">
+    <xacro:macro name="leg_joint" params="link_child name x y">
         <joint name="${name}" type="revolute">
             <origin xyz="0.0 0.0 0.0" rpy="0 0 0" />
-            <axis xyz = "1 0 0" />
+            <axis xyz = "0 1 0" />
             <parent link="base_link" />
             <child link="${link_child}" />
@@ -114,8 +114,8 @@
         </joint>
     </xacro:macro>
-    <xacro:macro name="foot_joint" params="link_parent link_child name">
+    <xacro:macro name="foot_joint" params="link_parent link_child name x y">
         <joint name="${name}" type="prismatic">
             <origin xyz="0.0 0.0 0.0" rpy="0 0 0" />
-            <axis xyz = "1 0 0" />
+            <axis xyz = "0 0 1" />
             <parent link="${link_parent}" />
             <child link="${link_child}" />
@@ -124,29 +124,39 @@
         </joint>
     </xacro:macro>
-    <xacro:leg leg_x="0" leg_y="0" name="leg_fl">
+    <!-- Xacro macros for our legs -->
+    <xacro:leg leg_x="${leg_fl_x}" leg_y="${leg_fl_y}" name="leg_fl">
     </xacro:leg>
-    <xacro:leg leg_x="0" leg_y="0" name="leg_fr">
+    <xacro:leg leg_x="${leg_fr_x}" leg_y="${leg_fr_y}" name="leg_fr">
     </xacro:leg>
-    <xacro:leg leg_x="0" leg_y="0" name="leg_rl">
+    <xacro:leg leg_x="${leg_rl_x}" leg_y="${leg_rl_y}" name="leg_rl">
     </xacro:leg>
-    <xacro:leg leg_x="0" leg_y="0" name="leg_rr">
+    <xacro:leg leg_x="${leg_rr_x}" leg_y="${leg_rr_y}" name="leg_rr">
     </xacro:leg>
-    <xacro:foot leg_x="0" leg_y="0" name="foot_rl">
+    <!-- Xacro macros for our feet -->
+    <xacro:foot leg_x="${leg_fl_x}" leg_y="${leg_fl_y}" name="foot_fl">
     </xacro:foot>
-    <xacro:foot leg_x="0" leg_y="0" name="foot_fr">
+    <xacro:foot leg_x="${leg_fr_x}" leg_y="${leg_fr_y}" name="foot_fr">
     </xacro:foot>
-    <xacro:foot leg_x="0" leg_y="0" name="foot_rl">
+    <xacro:foot leg_x="${leg_rl_x}" leg_y="${leg_rl_y}" name="foot_rl">
     </xacro:foot>
-    <xacro:foot leg_x="0" leg_y="0" name="foot_rr">
+    <xacro:foot leg_x="${leg_rr_x}" leg_y="${leg_rr_y}" name="foot_rr">
     </xacro:foot>
-    <xacro:leg_joint link_child="aa" name="aa">
+    <!-- Xacro macros for the links between our base link (the body) and the leg -->
+    <xacro:leg_joint link_child="leg_fl" name="base_to_leg_fl" x="${leg_fl_x}" y="${leg_fl_y}">
     </xacro:leg_joint>
-    <xacro:leg_joint link_child="aa" name="aa">
+    <xacro:leg_joint link_child="leg_fr" name="base_to_leg_fr" x="${leg_fr_x}" y="${leg_fr_y}">
     </xacro:leg_joint>
-    <xacro:leg_joint link_child="aa" name="aa">
+    <xacro:leg_joint link_child="leg_rl" name="base_to_leg_rl" x="${leg_rl_x}" y="${leg_rl_y}">
     </xacro:leg_joint>
-    <xacro:leg_joint link_child="aa" name="aa">
+    <xacro:leg_joint link_child="leg_rr" name="base_to_leg_rr" x="${leg_rr_x}" y="${leg_rr_y}">
     </xacro:leg_joint>
-    <xacro:foot_joint link_parent="aa" link_child="aa" name="aa">
+    <!-- Xacro macros for the links between our legs and our feet -->
+    <xacro:foot_joint link_parent="leg_fl" link_child="foot_fl" name="leg_to_foot_fl" x="${leg_fl_x}" y="${leg_fl_y}">
+    </xacro:foot_joint>
+    <xacro:foot_joint link_parent="leg_fr" link_child="foot_fr" name="leg_to_foot_fr" x="${leg_fr_x}" y="${leg_fr_y}">
+    </xacro:foot_joint>
+    <xacro:foot_joint link_parent="leg_rl" link_child="foot_rl" name="leg_to_foot_rl" x="${leg_rl_x}" y="${leg_rl_y}">
+    </xacro:foot_joint>
+    <xacro:foot_joint link_parent="leg_rr" link_child="foot_rr" name="leg_to_foot_rr" x="${leg_rr_x}" y="${leg_rr_y}">
     </xacro:foot_joint>
 </robot>

File: pmtg/gym-hsa_robot/gym_hsa_robot/resources/hsa_turtle_test.urdf (robot description, URDF)
Before this commit: robot hsa_robot, 8 links, 1 joints
Links:
- added link foot_fl, mass 0.02; collision box size=0.035 0.035 0.02; visual box size=0.035 0.035 0.02
Joints:
- removed joint aa
- added joint base_to_leg_fl: type revolute, parent base_link, child leg_fl, origin xyz=0.0 0.0 0.0 rpy=0 0 0, axis 1 0 0, limit lower=-0.785 upper=0.785 effort=10 velocity=1.0
- added joint base_to_leg_fr: type revolute, parent base_link, child leg_fr, origin xyz=0.0 0.0 0.0 rpy=0 0 0, axis 1 0 0, limit lower=-0.785 upper=0.785 effort=10 velocity=1.0
- added joint base_to_leg_rl: type revolute, parent base_link, child leg_rl, origin xyz=0.0 0.0 0.0 rpy=0 0 0, axis 1 0 0, limit lower=-0.785 upper=0.785 effort=10 velocity=1.0
- added joint base_to_leg_rr: type revolute, parent base_link, child leg_rr, origin xyz=0.0 0.0 0.0 rpy=0 0 0, axis 1 0 0, limit lower=-0.785 upper=0.785 effort=10 velocity=1.0
- added joint leg_to_foot_fl: type prismatic, parent leg_fl, child foot_fl, origin xyz=0.0 0.0 0.0 rpy=0 0 0, axis 1 0 0, limit lower=-0.785 upper=0.785 effort=10 velocity=1.0
- added joint leg_to_foot_fr: type prismatic, parent leg_fr, child foot_fr, origin xyz=0.0 0.0 0.0 rpy=0 0 0, axis 1 0 0, limit lower=-0.785 upper=0.785 effort=10 velocity=1.0
- added joint leg_to_foot_rl: type prismatic, parent leg_rl, child foot_rl, origin xyz=0.0 0.0 0.0 rpy=0 0 0, axis 1 0 0, limit lower=-0.785 upper=0.785 effort=10 velocity=1.0
- added joint leg_to_foot_rr: type prismatic, parent leg_rr, child foot_rr, origin xyz=0.0 0.0 0.0 rpy=0 0 0, axis 1 0 0, limit lower=-0.785 upper=0.785 effort=10 velocity=1.0

Commit message: xacro changes

File: pmtg/gym-hsa_robot/gym_hsa_robot/resources/hsa_turtle.xacro (robot description, xacro)
@@ -63,8 +63,8 @@
                 </geometry>
                 <material name="blue"/>
-                <origin rpy="0 0 0" xyz="leg_x leg_y -0.025"/>
+                <origin rpy="0 0 0" xyz="{leg_x} {leg_y} -0.025"/>
             </visual>
             <inertial>
-                <origin rpy="0 0 0" xyz="leg_x leg_y -0.025"/>
+                <origin rpy="0 0 0" xyz="${leg_x} ${leg_y} -0.025"/>
                 <mass value = "0.02"/>
                 <inertia ixx="${(1.0/12.0) * 0.02 * ( (0.035 * 0.035) + (0.05 * 0.05) ) }"
@@ -73,5 +73,5 @@
             </inertial>
             <collision>
-                <origin rpy="0 0 0" xyz="leg_x leg_y -0.025"/>
+                <origin rpy="0 0 0" xyz="${leg_x} ${leg_y} -0.025"/>
                 <geometry>
                     <box size="0.035 0.035 0.05" />
@@ -87,8 +87,8 @@
                 </geometry>
                 <material name="red"/>
-                <origin rpy="0 0 0" xyz="leg_x leg_y -0.06"/>
+                <origin rpy="0 0 0" xyz="${leg_x} ${leg_y} -0.06"/>
             </visual>
             <inertial>
-                <origin rpy="0 0 0" xyz="leg_x leg_y -0.06"/>
+                <origin rpy="0 0 0" xyz="${leg_x} ${leg_y} -0.06"/>
                 <mass value = "0.02"/>
                 <inertia ixx="${(1.0/12.0) * 0.02 * ( (0.035 * 0.035) + (0.02 * 0.02) ) }"
@@ -97,5 +97,5 @@
             </inertial>
             <collision>
-                <origin rpy="0 0 0" xyz="leg_x leg_y -0.06"/>
+                <origin rpy="0 0 0" xyz="${leg_x} ${leg_y} -0.06"/>
                 <geometry>
                     <box size="0.035 0.035 0.02" />
@@ -106,5 +106,5 @@
     <xacro:macro name="leg_joint" params="link_child name x y">
         <joint name="${name}" type="revolute">
-            <origin xyz="0.0 0.0 0.0" rpy="0 0 0" />
+            <origin xyz="${x} ${y} 0.0" rpy="0 0 0" />
             <axis xyz = "0 1 0" />
             <parent link="base_link" />
@@ -116,5 +116,5 @@
     <xacro:macro name="foot_joint" params="link_parent link_child name x y">
         <joint name="${name}" type="prismatic">
-            <origin xyz="0.0 0.0 0.0" rpy="0 0 0" />
+            <origin xyz="${x} ${y} -0.05" rpy="0 0 0" />
             <axis xyz = "0 0 1" />
             <parent link="${link_parent}" />

File: pmtg/gym-hsa_robot/gym_hsa_robot/resources/hsa_turtle_test.urdf (robot description, URDF)
Before this commit: robot hsa_robot, 9 links, 8 joints
Joints:
- joint base_to_leg_fl: axis 1 0 0 -> 0 1 0; origin xyz=0.0 0.0 0.0 rpy=0 0 0 -> xyz=0.035 0.06 0.0 rpy=0 0 0
- joint base_to_leg_fr: axis 1 0 0 -> 0 1 0; origin xyz=0.0 0.0 0.0 rpy=0 0 0 -> xyz=0.035 -0.06 0.0 rpy=0 0 0
- joint base_to_leg_rl: axis 1 0 0 -> 0 1 0; origin xyz=0.0 0.0 0.0 rpy=0 0 0 -> xyz=-0.035 0.06 0.0 rpy=0 0 0
- joint base_to_leg_rr: axis 1 0 0 -> 0 1 0; origin xyz=0.0 0.0 0.0 rpy=0 0 0 -> xyz=-0.035 -0.06 0.0 rpy=0 0 0
- joint leg_to_foot_fl: axis 1 0 0 -> 0 0 1; origin xyz=0.0 0.0 0.0 rpy=0 0 0 -> xyz=0.035 0.06 -0.05 rpy=0 0 0
- joint leg_to_foot_fr: axis 1 0 0 -> 0 0 1; origin xyz=0.0 0.0 0.0 rpy=0 0 0 -> xyz=0.035 -0.06 -0.05 rpy=0 0 0
- joint leg_to_foot_rl: axis 1 0 0 -> 0 0 1; origin xyz=0.0 0.0 0.0 rpy=0 0 0 -> xyz=-0.035 0.06 -0.05 rpy=0 0 0
- joint leg_to_foot_rr: axis 1 0 0 -> 0 0 1; origin xyz=0.0 0.0 0.0 rpy=0 0 0 -> xyz=-0.035 -0.06 -0.05 rpy=0 0 0

Commit message: urdf looking goodgit status

File: pmtg/gym-hsa_robot/gym_hsa_robot/resources/hsa_turtle.xacro (robot description, xacro)
@@ -4,4 +4,13 @@
      Date: 10/26/2022   -->
 <robot name="hsa_robot" xmlns:xacro="http://ros.org/wiki/xacro">
+    <material name="gray">
+	    <color rgba="0.5 0.5 0.5 1.0"/>
+	</material>
+    <material name="red">
+        <color rgba="0.8 0.0 0.0 1.0"/>
+    </material>
+    <material name="blue">
+        <color rgba="0.0 0.0 0.8 1.0"/>
+    </material>
 	<xacro:property name="torso_width" value="0.14" />
     <xacro:property name="torso_height" value="0.16" />
@@ -31,4 +40,6 @@
     <xacro:property name="foot_rr_x" value="0.4" />
     <xacro:property name="foot_rr_y" value="0.4" />
+    <link name="dummy">
+    </link>
 	<link name="base_link">
 		<visual>
@@ -36,7 +47,5 @@
 				<box size="${torso_width} ${torso_height} ${torso_depth}" />
 			</geometry>
-			<material name="gray">
-				<!-- color rgba="255 0 0 0.75" /-->
-			</material>
+            <material name="gray"/>
 			<origin rpy="0 0 0" xyz="0.0 0.0 0.0"/>
 		</visual>
@@ -47,5 +56,8 @@
 			<inertia ixx="${(1.0/12.0) * torso_mass * ( (torso_height * torso_height) + (torso_depth * torso_depth) ) }"
                                  iyy="${(1.0/12.0) * torso_mass * ( (torso_width * torso_width) + (torso_depth * torso_depth) ) }"
-                                 izz="${(1.0/12.0) * torso_mass * ( (torso_width * torso_width) + (torso_height * torso_height) ) }"/>
+                                 izz="${(1.0/12.0) * torso_mass * ( (torso_width * torso_width) + (torso_height * torso_height) ) }"
+                                 ixy="0"
+                                 ixz="0"
+                                 iyz="0"/>
     		</inertial>
 		<collision>
@@ -56,4 +68,8 @@
 		</collision>
     </link>
+    <joint name="dummy_joint" type="fixed">
+        <parent link="dummy"/>
+        <child link="base_link"/>
+    </joint>
     <xacro:macro name="leg" params="leg_x leg_y name">
         <link name="${name}">
@@ -63,5 +79,6 @@
                 </geometry>
                 <material name="blue"/>
-                <origin rpy="0 0 0" xyz="{leg_x} {leg_y} -0.025"/>
+                <origin rpy="0 0 0" xyz="0 0 -0.025"/>
+                <!-- <origin rpy="0 0 0" xyz="${leg_x} ${leg_y} -0.025"/> -->
             </visual>
             <inertial>
@@ -70,5 +87,8 @@
                 <inertia ixx="${(1.0/12.0) * 0.02 * ( (0.035 * 0.035) + (0.05 * 0.05) ) }"
                                  iyy="${(1.0/12.0) * 0.02 * ( (0.035 * 0.035) + (0.05 * 0.05) ) }"
-                                 izz="${(1.0/12.0) * 0.02 * ( (0.035 * 0.035) + (0.035 * 0.035) ) }"/>
+                                 izz="${(1.0/12.0) * 0.02 * ( (0.035 * 0.035) + (0.035 * 0.035) ) }"
+                                 ixy="0"
+                                 ixz="0"
+                                 iyz="0"/>
             </inertial>
             <collision>
@@ -87,12 +107,16 @@
                 </geometry>
                 <material name="red"/>
-                <origin rpy="0 0 0" xyz="${leg_x} ${leg_y} -0.06"/>
+                <origin rpy="0 0 0" xyz="0 0 0"/>
+                <!-- <origin rpy="0 0 0" xyz="${leg_x} ${leg_y} -0.06"/> -->
             </visual>
             <inertial>
                 <origin rpy="0 0 0" xyz="${leg_x} ${leg_y} -0.06"/>
-                <mass value = "0.02"/>
-                <inertia ixx="${(1.0/12.0) * 0.02 * ( (0.035 * 0.035) + (0.02 * 0.02) ) }"
-                                 iyy="${(1.0/12.0) * 0.02 * ( (0.035 * 0.035) + (0.02 * 0.02) ) }"
-                                 izz="${(1.0/12.0) * 0.02 * ( (0.035 * 0.035) + (0.035 * 0.035) ) }"/>
+                <mass value = "0.01"/>
+                <inertia ixx="${(1.0/12.0) * 0.01 * ( (0.035 * 0.035) + (0.01 * 0.01) ) }"
+                                 iyy="${(1.0/12.0) * 0.01 * ( (0.035 * 0.035) + (0.01 * 0.01) ) }"
+                                 izz="${(1.0/12.0) * 0.01 * ( (0.035 * 0.035) + (0.035 * 0.035) ) }"
+                                 ixy="0"
+                                 ixz="0"
+                                 iyz="0"/>
             </inertial>
             <collision>
@@ -106,20 +130,21 @@
     <xacro:macro name="leg_joint" params="link_child name x y">
         <joint name="${name}" type="revolute">
-            <origin xyz="${x} ${y} 0.0" rpy="0 0 0" />
-            <axis xyz = "0 1 0" />
+            <!-- <origin xyz="${x} ${y} 0.0" rpy="0 0 0" /> -->
+            <origin xyz="${x} ${y} -0.01" rpy="0 0 0" />
+            <axis xyz = "1 0 0" />
             <parent link="base_link" />
             <child link="${link_child}" />
                     <!-- What to set these to? -->
-            <limit velocity="1.0" effort="10" lower="${-1.57/2.0}" upper="${1.57/2.0}"/>
+            <limit velocity="1.0" effort="10" lower="-0.5" upper="0.5"/>
         </joint>
     </xacro:macro>
     <xacro:macro name="foot_joint" params="link_parent link_child name x y">
         <joint name="${name}" type="prismatic">
-            <origin xyz="${x} ${y} -0.05" rpy="0 0 0" />
+            <origin xyz="0.0 0.0 -0.06" rpy="0 0 0" />
             <axis xyz = "0 0 1" />
             <parent link="${link_parent}" />
             <child link="${link_child}" />
                     <!-- What to set these to? -->
-            <limit velocity="1.0" effort="10" lower="${-1.57/2.0}" upper="${1.57/2.0}"/>
+            <limit velocity="1.0" effort="10" lower="-0.02" upper="0.02"/>
         </joint>
     </xacro:macro>

File: pmtg/gym-hsa_robot/gym_hsa_robot/resources/hsa_turtle_test.urdf (robot description, URDF)
Before this commit: robot hsa_robot, 9 links, 8 joints
Links:
- added link dummy
- link foot_fl: mass 0.02 -> 0.01
- link foot_fr: mass 0.02 -> 0.01
- link foot_rl: mass 0.02 -> 0.01
- link foot_rr: mass 0.02 -> 0.01
Joints:
- added joint dummy_joint: type fixed, parent dummy, child base_link
- joint base_to_leg_fl: axis 0 1 0 -> 1 0 0; limit lower=-0.785 upper=0.785 effort=10 velocity=1.0 -> lower=-0.5 upper=0.5 effort=10 velocity=1.0; origin xyz=0.035 0.06 0.0 rpy=0 0 0 -> xyz=0.035 0.06 -0.01 rpy=0 0 0
- joint base_to_leg_fr: axis 0 1 0 -> 1 0 0; limit lower=-0.785 upper=0.785 effort=10 velocity=1.0 -> lower=-0.5 upper=0.5 effort=10 velocity=1.0; origin xyz=0.035 -0.06 0.0 rpy=0 0 0 -> xyz=0.035 -0.06 -0.01 rpy=0 0 0
- joint base_to_leg_rl: axis 0 1 0 -> 1 0 0; limit lower=-0.785 upper=0.785 effort=10 velocity=1.0 -> lower=-0.5 upper=0.5 effort=10 velocity=1.0; origin xyz=-0.035 0.06 0.0 rpy=0 0 0 -> xyz=-0.035 0.06 -0.01 rpy=0 0 0
- joint base_to_leg_rr: axis 0 1 0 -> 1 0 0; limit lower=-0.785 upper=0.785 effort=10 velocity=1.0 -> lower=-0.5 upper=0.5 effort=10 velocity=1.0; origin xyz=-0.035 -0.06 0.0 rpy=0 0 0 -> xyz=-0.035 -0.06 -0.01 rpy=0 0 0
- joint leg_to_foot_fl: limit lower=-0.785 upper=0.785 effort=10 velocity=1.0 -> lower=-0.02 upper=0.02 effort=10 velocity=1.0; origin xyz=0.035 0.06 -0.05 rpy=0 0 0 -> xyz=0.0 0.0 -0.06 rpy=0 0 0
- joint leg_to_foot_fr: limit lower=-0.785 upper=0.785 effort=10 velocity=1.0 -> lower=-0.02 upper=0.02 effort=10 velocity=1.0; origin xyz=0.035 -0.06 -0.05 rpy=0 0 0 -> xyz=0.0 0.0 -0.06 rpy=0 0 0
- joint leg_to_foot_rl: limit lower=-0.785 upper=0.785 effort=10 velocity=1.0 -> lower=-0.02 upper=0.02 effort=10 velocity=1.0; origin xyz=-0.035 0.06 -0.05 rpy=0 0 0 -> xyz=0.0 0.0 -0.06 rpy=0 0 0
- joint leg_to_foot_rr: limit lower=-0.785 upper=0.785 effort=10 velocity=1.0 -> lower=-0.02 upper=0.02 effort=10 velocity=1.0; origin xyz=-0.035 -0.06 -0.05 rpy=0 0 0 -> xyz=0.0 0.0 -0.06 rpy=0 0 0

Commit message: xacro looks great

File: pmtg/gym-hsa_robot/gym_hsa_robot/resources/hsa_turtle.xacro (robot description, xacro)
@@ -132,5 +132,5 @@
             <!-- <origin xyz="${x} ${y} 0.0" rpy="0 0 0" /> -->
             <origin xyz="${x} ${y} -0.01" rpy="0 0 0" />
-            <axis xyz = "1 0 0" />
+            <axis xyz = "0 1 0" />
             <parent link="base_link" />
             <child link="${link_child}" />
@@ -146,5 +146,5 @@
             <child link="${link_child}" />
                     <!-- What to set these to? -->
-            <limit velocity="1.0" effort="10" lower="-0.02" upper="0.02"/>
+            <limit velocity="1.0" effort="10" lower="-0.02" upper="0.0199"/>
         </joint>
     </xacro:macro>

File: pmtg/gym-hsa_robot/gym_hsa_robot/resources/hsa_turtle_test.urdf (robot description, URDF)
Before this commit: robot hsa_robot, 10 links, 9 joints
Joints:
- joint base_to_leg_fl: axis 1 0 0 -> 0 1 0
- joint base_to_leg_fr: axis 1 0 0 -> 0 1 0
- joint base_to_leg_rl: axis 1 0 0 -> 0 1 0
- joint base_to_leg_rr: axis 1 0 0 -> 0 1 0

Commit message: able to control joints in pybullet, joint limits and such seem to work as expected

File: pmtg/gym-hsa_robot/gym_hsa_robot/resources/hsa_turtle.xacro (robot description, xacro)
@@ -60,5 +60,5 @@
                                  ixz="0"
                                  iyz="0"/>
-    		</inertial>
+    	</inertial>
 		<collision>
       			<origin rpy="0 0 0" xyz="0.0 0.0 0.0"/>

Commit message: add inertia for dummy, doesn't freak out as much anymore. Not sure why legs aren't moving now

File: pmtg/gym-hsa_robot/gym_hsa_robot/resources/hsa_turtle.xacro (robot description, xacro)
@@ -41,4 +41,15 @@
     <xacro:property name="foot_rr_y" value="0.4" />
     <link name="dummy">
+        <inertial>
+      			<origin rpy="0 0 0" xyz="0.0 0.0 0.0"/>
+			<mass value = "0.001"/>
+			<!-- Fix the inertia tag-->
+			<inertia ixx="0"
+                     iyy="0"
+                     izz="0"
+                     ixy="0"
+                     ixz="0"
+                     iyz="0"/>
+    	</inertial>
     </link>
 	<link name="base_link">

File: pmtg/gym-hsa_robot/gym_hsa_robot/resources/hsa_turtle_test.urdf (robot description, URDF)
Before this commit: robot hsa_robot, 10 links, 9 joints
Links:
- link dummy: mass None -> 0.001
Joints:
- joint leg_to_foot_fl: limit lower=-0.02 upper=0.02 effort=10 velocity=1.0 -> lower=-0.02 upper=0.0199 effort=10 velocity=1.0
- joint leg_to_foot_fr: limit lower=-0.02 upper=0.02 effort=10 velocity=1.0 -> lower=-0.02 upper=0.0199 effort=10 velocity=1.0
- joint leg_to_foot_rl: limit lower=-0.02 upper=0.02 effort=10 velocity=1.0 -> lower=-0.02 upper=0.0199 effort=10 velocity=1.0
- joint leg_to_foot_rr: limit lower=-0.02 upper=0.02 effort=10 velocity=1.0 -> lower=-0.02 upper=0.0199 effort=10 velocity=1.0

Commit message: found appropriate trajectory generator, test_gym_install does orig gait

File: pmtg/gym-hsa_robot/gym_hsa_robot/resources/hsa_turtle.xacro (robot description, xacro)
@@ -147,5 +147,5 @@
             <child link="${link_child}" />
                     <!-- What to set these to? -->
-            <limit velocity="1.0" effort="10" lower="-0.5" upper="0.5"/>
+            <limit velocity="1.0" effort="10" lower="-0.3" upper="0.3"/>
         </joint>
     </xacro:macro>

Commit message: fixed some errors where I mixed up theta and epsilon

File: pmtg/gym-hsa_robot/gym_hsa_robot/resources/hsa_turtle.xacro (robot description, xacro)
@@ -16,5 +16,5 @@
     <xacro:property name="torso_height" value="0.16" />
     <xacro:property name="torso_depth" value="0.02" />
-    <xacro:property name="torso_mass" value="0.4" />
+    <xacro:property name="torso_mass" value="0.01" />
 	<xacro:property name="leg_length" value="0.4" />
 	<xacro:property name="leg_radius" value="0.025"/>

Commit message: made many changes. foremost, reduced leg swing period though allowed more general pmtg modifications to choose foot placement. should transfer better to real robot

File: pmtg/gym-hsa_robot/gym_hsa_robot/resources/hsa_turtle.xacro (robot description, xacro)
@@ -19,9 +19,9 @@
 	<xacro:property name="leg_length" value="0.4" />
 	<xacro:property name="leg_radius" value="0.025"/>
-	<xacro:property name="leg_mass" value="0.05" />
+	<xacro:property name="leg_mass" value="0.04" />
 	<xacro:property name="foot_width" value="0.1" />
     <xacro:property name="foot_height" value="0.1" />
     <xacro:property name="foot_depth" value="0.01" />
-	<xacro:property name="foot_mass" value="0.25" />
+	<xacro:property name="foot_mass" value="0.01" />
     <xacro:property name="leg_fl_x" value="0.035" />
     <xacro:property name="leg_fl_y" value="0.06" />

File: pmtg/gym-hsa_robot/gym_hsa_robot/resources/hsa_turtle_test.urdf (robot description, URDF)
Before this commit: robot hsa_robot, 10 links, 9 joints
Links:
- link foot_fl: mass 0.25 -> 0.01
- link foot_fr: mass 0.25 -> 0.01
- link foot_rl: mass 0.25 -> 0.01
- link foot_rr: mass 0.25 -> 0.01
