Commit message: testing more things looks better

File: pmtg/gym-hsa_robot/gym_hsa_robot/resources/hsa_turtle.xacro (robot description, xacro)
@@ -147,5 +147,5 @@
             <child link="${link_child}" />
                     <!-- What to set these to? -->
-            <limit velocity="1.0" effort="10" lower="-0.23" upper="0.23"/>
+            <limit velocity="1.0" effort="10" lower="-0.25" upper="0.25"/>
         </joint>
     </xacro:macro>
@@ -157,5 +157,5 @@
             <child link="${link_child}" />
                     <!-- What to set these to? -->
-            <limit velocity="1.0" effort="10" lower="-0.008" upper="0.0005"/>
+            <limit velocity="1.0" effort="10" lower="-0.008" upper="0.001"/>
         </joint>
     </xacro:macro>

Commit message: changes from past couple weeks. 1. imported lookup table into training, 2. applied gaussian noise as a percentage of total joint output, 3. limited output from legs by 20% as in real life

File: pmtg/gym-hsa_robot/gym_hsa_robot/resources/hsa_turtle.xacro (robot description, xacro)
@@ -146,6 +146,6 @@
             <parent link="base_link" />
             <child link="${link_child}" />
-                    <!-- What to set these to? -->
-            <limit velocity="1.0" effort="10" lower="-0.25" upper="0.25"/>
+                    <!-- Previously was +/-0.25, now we limited by 20% -->
+            <limit velocity="1.0" effort="10" lower="-0.2" upper="0.2"/>
         </joint>
     </xacro:macro>
@@ -156,6 +156,6 @@
             <parent link="${link_parent}" />
             <child link="${link_child}" />
-                    <!-- What to set these to? -->
-            <limit velocity="1.0" effort="10" lower="-0.008" upper="0.001"/>
+                    <!-- Previously was [-0.008, 0.001], now we limited by 20% -->
+            <limit velocity="1.0" effort="10" lower="-0.0064" upper="0.0008"/>
         </joint>
     </xacro:macro>
